File: Electronics/lcd13264-shield/lcd13264-shield.sch (EAGLE design)
At the start: 28 parts, among them J1 MICRO-SDCARD-CONNECTOR-330006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, Q1 PNP-500mA, U1 ARDUINO_SHIELDNO_SILK, X1 FH12-12S-1S, X2 FH12-12S-1S

Commit message: Routed baord. Need to put on finishing touches.
Parts:
- removed U1: ARDUINO_SHIELDNO_SILK, SparkFun-Boards:ARDUINO_SHIELDNO_SILK
- added J2: ARDUINO_R3_SHIELDUNO_R3_SHIELD_LOCK, SparkFun-Boards:ARDUINO_R3_SHIELDUNO_R3_SHIELD_LOCK
Connections:
- removed net N$11: U1.D8
- removed net N$12: U1.D7
- removed net N$13: U1.*D6
- removed net N$14: U1.*D5
- removed net N$15: U1.D4
- removed net N$26: U1.A0
- removed net N$27: U1.A1
- removed net N$28: U1.A2
- removed net N$29: U1.A3
- new net N$1: J2.IOREF
- new net SCL: J2.SCL
- new net SDA: J2.SDA
- net 3.3V: now also J2.3.3V, U2.OE, U3.OE; no longer U1.3.3V
- net 5V: now also J2.5V; no longer U1.5V
- net GND: now also J2.GND@0, J2.GND@1, J2.GND@2; no longer U1.GND@0, U1.GND@1, U1.GND@2
- net LCD_A0_5V: now also J2.*D9
- net LCD_BL_5V: now also J2.*D6; no longer U1.*D9
- net LCD_CS_5V: now also J2.D7
- net LCD_RST_5V: now also J2.D8
- net MISO_5V: now also J2.D12; no longer U1.D12
- net MOSI_5V: now also J2.*D11; no longer U1.*D11
- net N$16: now also J2.*D3; no longer U1.*D3
- net N$17: now also J2.D2; no longer U1.D2
- net N$20: now also J2.TX; no longer U1.TX
- net N$25: now also J2.RX; no longer U1.RX
- net N$31: now also J2.A4; no longer U1.A4
- net N$33: now also J2.A5; no longer U1.A5
- net N$34: now also J2.RES; no longer U1.RES
- net N$35: now also J2.VIN; no longer U1.VIN
- net N$36: now also J2.AREF; no longer U1.AREF
- net SCK_5V: now also J2.D13; no longer U1.D13
- net SD_CS_5V: now also J2.*D10; no longer U1.*D10
- net SW_A: now also J2.D4
- net SW_B: now also J2.*D5
- net SW_C: now also J2.A3
- net SW_D: now also J2.A2
- net SW_E: now also J2.A1
- net SW_F: now also J2.A0
